Commit message: Add 6DOF MoveIt arm bridge: ESP32 CAN firmware, 3 ROS2 bridge nodes, dummy test sketches; fix stuck TXERR, MCP2515 mode bug, LKTech TX contention

File: src/dicerox/dicerox_arm_urdf/urdf/Dicerox_robot_arm_URDF.xacro (robot description, xacro)
@@ -74,5 +74,5 @@
     <child link="Link2" />
     <axis xyz="0 0 1" />
-    <limit lower="-3.1416" upper="1.5708" effort="1000" velocity="1000" />
+    <limit lower="-3.14159" upper="0" effort="1000" velocity="1000" />
     <dynamics damping="0.1" friction="0.1" />
   </joint>
@@ -104,5 +104,5 @@
     <child link="Link3" />
     <axis xyz="0 0 1" />
-    <limit lower="-1.5708" upper="1.5708" effort="1000" velocity="1000" />
+    <limit lower="0" upper="3.49066" effort="1000" velocity="1000" />
     <dynamics damping="0.1" friction="0.1" />
   </joint>
